File: Domino Single Ethernet/Domino Single Ethernet Overlap No Teardrop.sch (EAGLE design)
At the start: 15 parts, among them J1 MH8-1, J3 B50(27-51)FP4-151-A613-B12, J5 MH18-1, J6 MH18-1

Commit message: Changed copyright
Other:
- note added: "The Domino Team may make changes to specifications and product"
- note added: "© 2014, The Domino Team All rights reserved."
- note removed: "Michel Stempin may make changes to specifications and product"
- note removed: "© 2014, Michel Stempin All rights reserved."
Changed lines of the file:
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@@
 <text x="302.26" y="12.7" size="0.8128" layer="94">Reference designs are provided "AS IS" and "WITH ALL FAULTS".</text>
 <text x="302.26" y="10.16" size="0.8128" layer="94">regarding this product, including but not limited to, any implied warranties of</text>
-<text x="302.26" y="6.35" size="0.8128" layer="94">Michel Stempin may make changes to specifications and product </text>
+<text x="302.26" y="6.35" size="0.8128" layer="94">The Domino Team may make changes to specifications and product </text>
 <text x="302.26" y="11.43" size="0.8128" layer="94">Global Marine Networks disclaims all other warranties express or implied, </text>
 <text x="302.26" y="8.89" size="0.8128" layer="94">merchantibility or fitness for any particular application.</text>
@@
 <text x="256.54" y="7.62" size="1.778" layer="94" align="center">Domino
 Qi</text>
-<text x="345.44" y="20.32" size="1.27" layer="94">© 2014, Michel Stempin
+<text x="345.44" y="20.32" size="1.27" layer="94">© 2014, The Domino Team
 All rights reserved.</text>
 <text x="379.222" y="5.334" size="1.778" layer="94">&gt;REV</text>
