File: Domino USB MicroSD/Domino USB MicroSD No Teardrop.sch (EAGLE design)
At the start: 69 parts, among them J1 MH5-2-0.1, J2 MH4-1, U1 MP65150DJ, U2 AU6350-MGL, Y1 12 MHz

Commit message: Changed copyright
Other:
- note added: "The Domino Team may make changes to specifications and product"
- note added: "© 2014, The Domino Team All rights reserved."
- note removed: "Michel Stempin may make changes to specifications and product"
- note removed: "© 2014, Michel Stempin All rights reserved."
Changed lines of the file:
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@@
 <layer number="102" name="CC-BY-SA_Letters" color="0" fill="4" visible="yes" active="yes"/>
 <layer number="103" name="CC-BY-SA_Filling" color="15" fill="1" visible="yes" active="yes"/>
+<layer number="107" name="legend" color="7" fill="1" visible="yes" active="yes"/>
+<layer number="108" name="Module_Measures" color="7" fill="1" visible="yes" active="yes"/>
 <layer number="119" name="mUnrouted" color="7" fill="1" visible="no" active="no"/>
 <layer number="126" name="mbNames" color="7" fill="1" visible="no" active="no"/>
@@
 <text x="302.26" y="12.7" size="0.8128" layer="94">Reference designs are provided "AS IS" and "WITH ALL FAULTS".</text>
 <text x="302.26" y="10.16" size="0.8128" layer="94">regarding this product, including but not limited to, any implied warranties of</text>
-<text x="302.26" y="6.35" size="0.8128" layer="94">Michel Stempin may make changes to specifications and product </text>
+<text x="302.26" y="6.35" size="0.8128" layer="94">The Domino Team may make changes to specifications and product </text>
 <text x="302.26" y="11.43" size="0.8128" layer="94">Global Marine Networks disclaims all other warranties express or implied, </text>
 <text x="302.26" y="8.89" size="0.8128" layer="94">merchantibility or fitness for any particular application.</text>
@@
 <text x="256.54" y="7.62" size="1.778" layer="94" align="center">Domino
 Qi</text>
-<text x="345.44" y="20.32" size="1.27" layer="94">© 2014, Michel Stempin
+<text x="345.44" y="20.32" size="1.27" layer="94">© 2014, The Domino Team
 All rights reserved.</text>
 <text x="379.222" y="5.334" size="1.778" layer="94">&gt;REV</text>
