File: Domino USB MicroSD/Domino USB MicroSD Passive Overcurrent Protection.brd (EAGLE design)
At the start: 27.9 x 10.2 mm, 51 parts, among them J1 MH5-2-0.1, J2 MH4-1, U1 AU6350-MGL, Y1 12 MHz

Commit message: Changed copyright
Other:
- board text added: "Reference designs are provided "AS IS" and "WITH ALL FAULTS". The Domino Team disclaims all other warranties express or implied, regarding this product, including but not limited to, any implied warranties of merchantibility or fitness for any particular application."
- board text added: "The Domino Team may make changes to specifications and product descriptions at any time, without notice."
- board text added: "© 2014, The Domino Team All rights reserved."
- board text removed: "Michel Stempin may make changes to specifications and product descriptions at any time, without notice."
- board text removed: "Reference designs are provided "AS IS" and "WITH ALL FAULTS". Michel Stempin disclaims all other warranties express or implied, regarding this product, including but not limited to, any implied warranties of merchantibility or fitness for any particular application."
- board text removed: "© 2014, Michel Stempin. All rights reserved."
Changed lines of the file:
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@@
 See creativecommons.org/licenses/by-sa/4.0/</text>
 <text x="34.29" y="-51.943" size="0.8128" layer="48" ratio="20">Reference designs are provided "AS IS" and "WITH ALL FAULTS".
-Michel Stempin disclaims all other warranties express or implied,
+The Domino Team disclaims all other warranties express or implied,
 regarding this product, including but not limited to, any implied warranties of
 merchantibility or fitness for any particular application.</text>
-<text x="34.29" y="-55.753" size="0.8128" layer="48" ratio="20">Michel Stempin may make changes to specifications and product descriptions
+<text x="34.29" y="-55.753" size="0.8128" layer="48" ratio="20">The Domino Team may make changes to specifications and product descriptions
 at any time, without notice.</text>
-<text x="74.93" y="-41.91" size="1.27" layer="48" ratio="20">© 2014, Michel Stempin.
+<text x="74.93" y="-41.91" size="1.27" layer="48" ratio="20">© 2014, The Domino Team
 All rights reserved.</text>
 <text x="115.57" y="-57.15" size="1.778" layer="48">Rev.</text>
