File: Domino Qi/Domino Qi.brd (EAGLE design)
At the start: 68.6 x 53.3 mm, 128 parts, among them J1 MH5-2-0.1, J2 MH4-1, J3 B50(27-51)FP4-151-A613-B12, J4 FR04-2, J6 MH6-1, M2 DOMINO, SW1 IT-1124SMD, U12 NTB0104GU12, U13 NTB0102GF, U2 MP2162GQH, U3 AU6350-MGL, U4 MP65150DJ, U5 MAX3375EEKA+T, Y1 12 MHz

Commit message: Changed copyright
Other:
- board text added: "Reference designs are provided "AS IS" and "WITH ALL FAULTS". The Domino Team disclaims all other warranties express or implied, regarding this product, including but not limited to, any implied warranties of merchantibility or fitness for any particular application."
- board text added: "The Domino Team may make changes to specifications and product descriptions at any time, without notice."
- board text added: "© 2014, The Domino Team. All rights reserved."
- board text removed: "Michel Stempin may make changes to specifications and product descriptions at any time, without notice."
- board text removed: "Reference designs are provided "AS IS" and "WITH ALL FAULTS". Michel Stempin disclaims all other warranties express or implied, regarding this product, including but not limited to, any implied warranties of merchantibility or fitness for any particular application."
- board text removed: "© 2014, Michel Stempin. All rights reserved."
Changed lines of the file:
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@@
 See creativecommons.org/licenses/by-sa/4.0/</text>
 <text x="52.07" y="-38.1" size="0.8128" layer="48" ratio="20">Reference designs are provided "AS IS" and "WITH ALL FAULTS".
-Michel Stempin disclaims all other warranties express or implied,
+The Domino Team disclaims all other warranties express or implied,
 regarding this product, including but not limited to, any implied warranties of
 merchantibility or fitness for any particular application.</text>
-<text x="52.07" y="-41.91" size="0.8128" layer="48" ratio="20">Michel Stempin may make changes to specifications and product descriptions
+<text x="52.07" y="-41.91" size="0.8128" layer="48" ratio="20">The Domino Team may make changes to specifications and product descriptions
 at any time, without notice.</text>
-<text x="92.71" y="-27.94" size="1.27" layer="48" ratio="20">© 2014, Michel Stempin.
+<text x="92.71" y="-27.94" size="1.27" layer="48" ratio="20">© 2014, The Domino Team.
 All rights reserved.</text>
 <text x="97.79" y="10.16" size="1.27" layer="48" ratio="10">NOTES:</text>

Commit message: Work in progress: changed for PCB antenna and removed Schottky diode on Domino Qi Mini, first Domino Qi draft
Parts:
- removed A1: ACA-5036-A2-CC-S, Domino:ACA-5036-A2-CC-S
- removed C15: 22u, Domino:C0805
- removed C16: 10p, Domino:C0402
- removed C17, C31, C32, C33, C36, C41, C42, C43, C44, C48, C49: 100n, Domino:C0402
- removed C19, C21: DNP, Domino:C0402
- removed C20: 10n, Domino:C0402
- removed C34: 2n2, Domino:C1206
- removed C35: 1n, Domino:C1206
- removed C37: 10u, Domino:C0805
- removed D1: MBRM130LT1G, Domino:DO-216AA
- removed D3: RED, Domino:LED0603
- removed D4: BLUE, Domino:LED0603
- removed F3: 0ZCG0110FF2C, Domino:PTC1812
- removed J3: B50(27-51)FP4-151-A613-B12, Domino:B50(27-51)FP4-151-A613-B12
- removed J4: FR04-2, Domino:FR04-2-0.1
- removed J6: MH6-1, Domino:MH6-1-0.1
- removed L2: SWPA252012S1R0NT, Domino:SWPA252012S
- removed L4: BLM31PG601SN1L, Domino:FB1206
- removed M2: DOMINO, Domino:DOMINO
- removed R10, R9: 0R, Domino:R0603
- removed R11: 270R, Domino:R0603
- removed R12, R13: 0R, Domino:R0402
- removed R14: 1k, Domino:R0402
- removed R15: 10k, Domino:R0402
- removed R42, R43, R44, R45: 49R9, Domino:R0402
- removed S1: USB_MR5-003A, Domino:USB_MR5-003A
- removed SW1: IT-1124SMD, Domino:IT-1124SMD
- removed U12: NTB0104GU12, Domino:XQFN-12
- removed U13: NTB0102GF, Domino:SOT1089
- removed U2: MP2162GQH, Domino:QFN-8_2X1.5
- removed U5: MAX3375EEKA+T, Domino:SOT23-8
- added J8: 11A009-1702-00, Domino:11A009-1702-00
- added M1: DOMINO_QI_MINI, Domino:DOMINO_QI_MINI
- added U$13: DOMINO_QI_LOGO, Domino:DOMINO_QI_LOGO
- C13: value 22u -> 2n2; device Domino:C0805 -> Domino:C1206
- C2: value 22u -> 100n; device Domino:C1206 -> Domino:C0402
- C3: value 10p -> 2n2; device Domino:C0402 -> Domino:C1206
- C7: value 22p -> 100n
- R1: value 10k -> 49R9
- R2: value 33k2 -> 49R9
- R3: value 150k -> 49R9
- R8: value 270R -> 49R9
- moved C1 281.5 mm to (69.4, 79.0)
- moved C10 281.5 mm to (97.4, 79.0)
- moved C11 281.5 mm to (49.4, 73.0)
- moved C12 281.5 mm to (50.4, 79.0)
- moved C14 281.5 mm to (77.4, 79.0)
- moved C18 281.5 mm to (55.4, 79.0)
- moved C22 281.5 mm to (60.4, 79.0)
- moved C23 281.5 mm to (65.4, 79.0)
- moved C24 281.5 mm to (52.4, 73.0)
- moved C25 281.5 mm to (55.4, 73.0)
- moved C26 281.5 mm to (89.4, 79.0)
- moved C28 281.5 mm to (58.4, 73.0)
- moved C29 281.5 mm to (61.4, 73.0)
- moved C30 281.5 mm to (64.4, 73.0)
- moved C4 281.5 mm to (85.4, 68.0)
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Connections:
- removed net !RESET_L: M2.4
- removed net +2.5VD_OUT: M2.23, R10.2
- removed net +2V5: C43.2, C44.2, C48.2, R10.1, R14.2, U12.1, U12.12, U13.3, U13.6, U5.3
- removed net +3.3VD_IN1: M2.25, M2.26, R8.2, R9.2
- removed net +VIO: C41.1, C42.1, C49.1, U12.11, U13.7, U5.7
- removed net +VUSB: D1.2, L4.1
- removed net ANT0: M2.59, R12.1
- removed net ANT0_50R: A1.FEED, C21.1, R13.2
- removed net ANT0_EXT: C19.1, R12.2, R13.1
- removed net BLUE_LED: D4.2, R11.1
- removed net EN: R1.2, U2.1
- removed net FB: C7.1, R2.2, R3.2, U2.2
- removed net FLASH_WP: M2.50
- removed net GPIO24: M2.28
- removed net I2S_CK: M2.34
- removed net I2S_MCK: M2.31
- removed net I2S_MICIN: M2.30
- removed net I2S_SD: M2.32
- removed net I2S_WS: M2.33
- removed net IOREF: BOARD1.IOREF
- removed net JTAG_TCK: M2.7
- removed net JTAG_TDI: M2.8
- removed net JTAG_TDO: M2.9
- removed net JTAG_TMS: M2.6
- removed net JUMPSTART: R14.1, SW1.1
- removed net LED0: M2.19, R11.2
- removed net LED1: M2.18
- removed net LED2: M2.17
- removed net LED3: M2.16
- removed net LED4: M2.15
- removed net LED5: M2.14
- removed net LED6: M2.13
- removed net LED7: M2.12
- removed net LED8: M2.11
- removed net N$1: D3.2, R8.1
- removed net N$2: U12.5
- removed net N$3: U12.4
- removed net N$4: U12.3
- removed net N$5: U12.2
- removed net N$6: U12.10
- removed net N$7: U12.9
- removed net N$8: U12.8
- removed net N$9: U12.7
- removed net P0_RX+: M2.41
- removed net P0_RX-: M2.42
- removed net P0_TX+: M2.43
- removed net P0_TX-: M2.44
- removed net P4_LED_L_A: J3.13, J4.6
- removed net P4_LED_L_C: J3.14, J4.8
- removed net P4_LED_R_A: J3.11, J4.2
- removed net P4_LED_R_C: J3.12, J4.4
- removed net P4_RX+: M2.36
- removed net P4_RX-: M2.37
- removed net P4_TX+: M2.38
- removed net P4_TX-: M2.39
- removed net PE: C35.1, S1.S$1, S1.S$2, S1.S$3
- removed net SPDIF_OUT: M2.29
- removed net SPI_CLK: M2.46
- removed net SPI_CS: M2.48
- removed net SPI_MISO: M2.49
- removed net SPI_MOSI: M2.47
- removed net SW: L2.1, U2.6
- removed net UART_CTS: M2.56
- removed net UART_RTS: C20.1, M2.55, R15.2, SW1.3
- removed net UART_RX: M2.20
- removed net UART_TX: M2.21
- removed net VBUS: C36.1, C37.1, F3.2, S1.1
- removed net VC12: J3.9, J4.5
- removed net VC36: J3.10, J4.7
- removed net VC45: J3.4, J4.1
- removed net VC78: J3.5, J4.3
- removed net VPROT: F3.1, L4.2
- removed net XLNA: M2.5
- new net !RESET: BOARD1.5, BOARD1.RESET$1, M1.27
- new net 3V3: BOARD1.3V3
- new net 3V3@1: M1.32
- new net 3V3@2: M1.13
- new net A0: BOARD1.A0, M1.1
- new net A1: BOARD1.A1, M1.2
- new net A2: BOARD1.A2, M1.9
- new net A3: BOARD1.A3, M1.10
- new net A4: BOARD1.A4, M1.11
- new net A5: BOARD1.A5, M1.12
- new net AREF: BOARD1.AREF, M1.43
- new net D4: BOARD1.D4, M1.29
- new net D5: BOARD1.D5, M1.30
- new net D6: BOARD1.D6, M1.31
- new net GP6: M1.42
- new net HANDSHAKE: BOARD1.D7, M1.34
- new net IO10: BOARD1.D10, M1.37
- new net IO11: BOARD1.D11, M1.38
- new net IO12: BOARD1.D12, M1.39
- new net IO13: BOARD1.D13, M1.41
- new net IO8: BOARD1.D8, M1.35
- new net IO9: BOARD1.D9, M1.36
- new net MISO: BOARD1.1, M1.17
- new net MOSI: BOARD1.4, M1.15
- new net RXD1: BOARD1.D0, M1.24
- new net SCK: BOARD1.3, M1.14
- new net SCL: BOARD1.D3, BOARD1.SCL, M1.28
- new net SDA: BOARD1.D2, BOARD1.SDA, M1.26
- new net SS: M1.16
- new net TXD1: BOARD1.D1, M1.25
- net +2VA_ETH_OUT: now also C7.2, J8.4, J8.5, M1.8; no longer C33.2, J3.3, J6.6, M2.40
- net +3V3: no longer C13.1, C15.1, C16.1, C17.1, C7.2, L2.2, M2.24, R3.1, R9.1, U2.4
- net +5V: no longer C2.1, C3.1, C5.1, D1.1, R1.1, U2.7
- net 5V: now also BOARD1.IOREF, M1.19
- net GND: now also BOARD1.GND$1, BOARD1.GND$2, C13.1, C2.1, C3.1, C5.1, C7.1, M1.18, M1.22, M1.23, M1.3, M1.33, M1.44; no longer A1.GND$1, A1.GND$2, C13.2, C15.2, C16.2, C17.2, C19.2, C2.2, C20.2, C21.2, C3.2, C31.1, C32.1, C33.1, C34.1, C35.2, C36.2, C37.2, C41.2, C42.2, C43.1, C44.1, C48.1, C49.2, C5.2, D3.1, D4.1, J6.1, M2.1, M2.10, M2.2, M2.22, M2.27, M2.3, M2.35, M2.45, M2.51, M2.54, M2.57, M2.58, M2.60, R15.1, R2.1, S1.5, U12.6, U13.2, U2.3, U2.5, U5.2
- net P4_RX: now also C5.2, R1.1, R3.1; no longer C31.2, R42.1, R43.1
- net P4_RX_N: now also J8.6, M1.5, R1.2; no longer J3.8, J6.3, R43.2
- net P4_RX_P: now also J8.3, M1.4, R3.2; no longer J3.7, J6.2, R42.2
- net P4_TX: now also C2.2, R2.1, R8.1; no longer C32.2, R44.1, R45.1
- net P4_TX_N: now also J8.2, M1.7, R8.2; no longer J3.2, J6.5, R45.2
- net P4_TX_P: now also J8.1, M1.6, R2.2; no longer J3.1, J6.4, R44.2
- net SHIELD: now also C13.2, C3.2, J8.8, J8.SH$1, J8.SH$2; no longer C34.2, J3.6, J3.SH$1, J3.SH$2
- net USB_N: now also M1.20; no longer M2.52
- net USB_P: now also M1.21; no longer M2.53
- net VIN: now also M1.40
