File: Domino Qi/Domino Qi.sch (EAGLE design)
At the start: 126 parts, among them J1 MH5-2-0.1, J2 MH4-1, J3 B50(27-51)FP4-151-A613-B12, J4 FR04-2, J6 MH6-1, M2 DOMINO, SW1 IT-1124SMD, U12 NTB0104GU12, U13 NTB0102GF, U2 MP2162GQH, U3 AU6350-MGL, U4 MP65150DJ, U5 MAX3375EEKA+T, Y1 12 MHz

Commit message: Changed copyright
Other:
- note added: "© 2014, The Domino Team All rights reserved."
- note removed: "© 2014, Michel Stempin All rights reserved."
Changed lines of the file:
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@@
 <layer number="102" name="CC-BY-SA_Letters" color="0" fill="4" visible="yes" active="yes"/>
 <layer number="103" name="CC-BY-SA_Filling" color="15" fill="1" visible="yes" active="yes"/>
+<layer number="107" name="legend" color="7" fill="1" visible="yes" active="yes"/>
+<layer number="108" name="Module_Measures" color="7" fill="1" visible="yes" active="yes"/>
 <layer number="119" name="mUnrouted" color="7" fill="1" visible="no" active="no"/>
 <layer number="126" name="mbNames" color="7" fill="1" visible="no" active="no"/>
@@
 <text x="480.06" y="8.89" size="0.8128" layer="94">merchantibility or fitness for any particular application.</text>
 <text x="480.06" y="5.08" size="0.8128" layer="94">descriptions at any time, without notice.</text>
-<text x="523.24" y="20.32" size="1.27" layer="94">© 2014, Michel Stempin
+<text x="523.24" y="20.32" size="1.27" layer="94">© 2014, The Domino Team
 All rights reserved.</text>
 <text x="557.022" y="5.334" size="1.778" layer="94">&gt;REV</text>

Commit message: Work in progress: changed for PCB antenna and removed Schottky diode on Domino Qi Mini, first Domino Qi draft
Parts:
- removed A1: ACA-5036-A2-CC-S, Domino:ACA-5036-A2-CC-S
- removed C15: 22u, Domino:CAP_0805
- removed C16: 10p, Domino:CAP_0402
- removed C17, C31, C32, C33, C36, C41, C42, C43, C44, C48, C49: 100n, Domino:CAP_0402
- removed C19, C21: DNP, Domino:CAP_0402
- removed C20: 10n, Domino:CAP_0402
- removed C34: 2n2, Domino:CAP_1206
- removed C35: 1n, Domino:CAP_1206
- removed C37: 10u, Domino:CAP_0805
- removed D1: MBRM130LT1G, Domino:MBRM130LT1G
- removed D3: RED, Domino:LED_0603
- removed D4: BLUE, Domino:LED_0603
- removed F3: 0ZCG0110FF2C, Domino:0ZCG0110FF2C
- removed J3: B50(27-51)FP4-151-A613-B12, Domino:B50(27-51)FP4-151-A613-B12
- removed J4: FR04-2, Domino:FR04-2
- removed J6: MH6-1, Domino:MH6-1
- removed L2: SWPA252012S1R0NT, Domino:SWPA252012S1R0NT
- removed L4: BLM31PG601SN1L, Domino:FB_1206
- removed M2: DOMINO, Domino:DOMINO
- removed R10, R9: 0R, Domino:RES_0603
- removed R11: 270R, Domino:RES_0603
- removed R12, R13: 0R, Domino:RES_0402
- removed R14: 1k, Domino:RES_0402
- removed R15: 10k, Domino:RES_0402
- removed R42, R43, R44, R45: 49R9, Domino:RES_0402
- removed S1: USB_MR5-003A, Domino:USB_MR5-003A
- removed SW1: IT-1124SMD, Domino:IT-1124SMD
- removed U12: NTB0104GU12, Domino:NTB0104GU12
- removed U13: NTB0102GF, Domino:NTB0102GF
- removed U2: MP2162GQH, Domino:MP2162GQH
- removed U5: MAX3375EEKA+T, Domino:MAX3375EEKA+T
- added J8: 11A009-1702-00, Domino:11A009-1702-00
- added M1: DOMINO_QI_MINI, Domino:DOMINO_QI_MINI
- added U$13: DOMINO_QI_LOGO, Domino:DOMINO_QI_LOGO
- C13: value 22u -> 2n2; device Domino:CAP_0805 -> Domino:CAP_1206; PARTNO C0805_22u_X5R_20%_CER_6V3 -> C1210_2n2_X7R_10%_CER_2kV; TC X5R -> X7R; TOL ±20% -> ±10%; VOLT 6.3V -> 2kV
- C2: value 22u -> 100n; device Domino:CAP_1206 -> Domino:CAP_0402; PARTNO C1206_22u_X7R_20%_CER_10V -> C0402_100n_X7R_10%_CER_50V; TOL ±20% -> ±10%; VOLT 10V -> 50V
- C3: value 10p -> 2n2; device Domino:CAP_0402 -> Domino:CAP_1206; PARTNO C0402_10p_NP0_5%_CER_50V -> C1210_2n2_X7R_10%_CER_2kV; TC NP0 -> X7R; TOL ±5% -> ±10%; VOLT 50V -> 2kV
- C7: value 22p -> 100n; PARTNO C0402_22p_NP0_5%_CER_50V -> C0402_100n_X7R_10%_CER_50V; TC NP0 -> X7R; TOL ±5% -> ±10%
- R1: value 10k -> 49R9; PARTNO R0402_10k_5%_62.5mW -> R0402_49R9_1%_62.5mW; TOL 5% -> 1%
- R2: value 33k2 -> 49R9; PARTNO R0402_33k2_1%_62.5mW -> R0402_49R9_1%_62.5mW
- R3: value 150k -> 49R9; PARTNO R0402_150k_1%_62.5mW -> R0402_49R9_1%_62.5mW
- R8: value 270R -> 49R9; PARTNO R0402_270R_5%_62.5mW -> R0402_49R9_1%_62.5mW; TOL 5% -> 1%
Connections:
- removed net !RESET_L: M2.!RESET_L
- removed net +2.5VD_OUT: M2.+2.5VD_OUT, R10.2
- removed net +2V5: C43.2, C44.2, C48.2, R10.1, R14.2, U12.OE, U12.VCCA, U13.OE, U13.VCCA, U5.VL
- removed net +3.3VD_IN1: M2.+3.3VD_IN@1, M2.+3.3VD_IN@2, R8.2, R9.2
- removed net +VIO: C41.1, C42.1, C49.1, U12.VCCB, U13.VCCB, U5.VCC
- removed net +VUSB: D1.A, L4.1
- removed net ANT0: M2.ANT0, R12.1
- removed net ANT0_50R: A1.A, C21.1, R13.2
- removed net ANT0_EXT: C19.1, R12.2, R13.1
- removed net BLUE_LED: D4.A, R11.1
- removed net EN: R1.2, U2.EN
- removed net FB: C7.1, R2.2, R3.2, U2.FB
- removed net FLASH_WP: M2.FLASH_WP
- removed net GPIO24: M2.GPIO24
- removed net I2S_CK: M2.I2S_CK
- removed net I2S_MCK: M2.I2S_MCK
- removed net I2S_MICIN: M2.I2S_MICIN
- removed net I2S_SD: M2.I2S_SD
- removed net I2S_WS: M2.I2S_WS
- removed net JTAG_TCK: M2.JTAG_TCK
- removed net JTAG_TDI: M2.JTAG_TDI
- removed net JTAG_TDO: M2.JTAG_TDO
- removed net JTAG_TMS: M2.JTAG_TMS
- removed net JUMPSTART: R14.1, SW1.1
- removed net LED0: M2.LED0, R11.2
- removed net LED1: M2.LED1
- removed net LED2: M2.LED2
- removed net LED3: M2.LED3
- removed net LED4: M2.LED4
- removed net LED5: M2.LED5
- removed net LED6: M2.LED6
- removed net LED7: M2.LED7
- removed net LED8: M2.LED8
- removed net N$1: D3.A, R8.1
- removed net N$2: U12.A4
- removed net N$3: U12.A3
- removed net N$4: U12.A2
- removed net N$5: U12.A1
- removed net N$6: U12.B1
- removed net N$7: U12.B2
- removed net N$8: U12.B3
- removed net N$9: U12.B4
- removed net P0_RX+: M2.P0_RX+
- removed net P0_RX-: M2.P0_RX-
- removed net P0_TX+: M2.P0_TX+
- removed net P0_TX-: M2.P0_TX-
- removed net P4_LED_L_A: J3.13, J4.6
- removed net P4_LED_L_C: J3.14, J4.8
- removed net P4_LED_R_A: J3.11, J4.2
- removed net P4_LED_R_C: J3.12, J4.4
- removed net P4_RX+: M2.P4_RX+
- removed net P4_RX-: M2.P4_RX-
- removed net P4_TX+: M2.P4_TX+
- removed net P4_TX-: M2.P4_TX-
- removed net PE: C35.1, S1.M0, S1.M1, S1.M2
- removed net SPDIF_OUT: M2.SPDIF_OUT
- removed net SPI_CLK: M2.SPI_CLK
- removed net SPI_CS: M2.SPI_CS
- removed net SPI_MISO: M2.SPI_MISO
- removed net SPI_MOSI: M2.SPI_MOSI
- removed net SW: L2.1, U2.SW
- removed net UART_CTS: M2.UART_CTS
- removed net UART_RTS: C20.1, M2.UART_RTS, R15.2, SW1.3
- removed net UART_RX: M2.UART_RX
- removed net UART_TX: M2.UART_TX
- removed net VBUS: C36.1, C37.1, F3.2, S1.1
- removed net VC12: J3.9, J4.5
- removed net VC36: J3.10, J4.7
- removed net VC45: J3.4, J4.1
- removed net VC78: J3.5, J4.3
- removed net VPROT: F3.1, L4.2
- removed net XLNA: M2.XLNA
- new net !RESET: BOARD1.RESET@1, BOARD1.RESET@2, M1.!RESET
- new net 3V3: BOARD1.3V3
- new net 3V3@1: M1.3V3@1
- new net 3V3@2: M1.3V3@2
- new net 5V: BOARD1.5V@1, BOARD1.5V@2, BOARD1.IOREF, M1.5V
- new net A0: BOARD1.A0, M1.A0
- new net A1: BOARD1.A1, M1.A1
- new net A2: BOARD1.A2, M1.A2
- new net A3: BOARD1.A3, M1.A3
- new net A4: BOARD1.A4, M1.A4
- new net A5: BOARD1.A5, M1.A5
- new net AREF: BOARD1.AREF, M1.AREF
- new net D4: BOARD1.D4, M1.D4
- new net D5: BOARD1.D5, M1.D5
- new net D6: BOARD1.D6, M1.D6
- new net GP6: M1.GP6
- new net HANDSHAKE: BOARD1.D7, M1.HANDSHAKE
- new net IO10: BOARD1.D10, M1.IO10
- new net IO11: BOARD1.D11, M1.IO11
- new net IO12: BOARD1.D12, M1.IO12
- new net IO13: BOARD1.D13, M1.IO13
- new net IO8: BOARD1.D8, M1.IO8
- new net IO9: BOARD1.D9, M1.IO9
- new net MISO: BOARD1.MISO, M1.MISO
- new net MOSI: BOARD1.MOSI, M1.MOSI
- new net RXD1: BOARD1.D0(RX0), M1.RXD1
- new net SCK: BOARD1.SCK, M1.SCK
- new net SCL: BOARD1.D3, BOARD1.SCL, M1.SCL
- new net SDA: BOARD1.D2, BOARD1.SDA, M1.SDA
- new net SS: M1.SS
- new net TXD1: BOARD1.D1(TX0), M1.TXD1
- new net VIN: BOARD1.VIN, M1.VIN
- net +2VA_ETH_OUT: now also C7.2, J8.P4, J8.P5, M1.+2VA_ETH_OUT; no longer C33.2, J3.3, J6.6, M2.+2VA_ETH_OUT
- net +3V3: no longer C13.1, C15.1, C16.1, C17.1, C7.2, L2.2, M2.+3.3VD_FLASH_IN, R3.1, R9.1, U2.OUT
- net +5V: no longer C2.1, C3.1, C5.1, D1.C, R1.1, U2.VIN
- net GND: now also BOARD1.GND@1, BOARD1.GND@2, BOARD1.GND@3, BOARD1.GND@4, C13.1, C2.1, C3.1, C5.1, C7.1, M1.GND@1, M1.GND@2, M1.GND@3, M1.GND@4, M1.GND@5, M1.GND@6; no longer A1.GND@1, A1.GND@2, C13.2, C15.2, C16.2, C17.2, C19.2, C2.2, C20.2, C21.2, C3.2, C31.1, C32.1, C33.1, C34.1, C35.2, C36.2, C37.2, C41.2, C42.2, C43.1, C44.1, C48.1, C49.2, C5.2, D3.C, D4.C, J6.1, M2.GND@10, M2.GND@11, M2.GND@13, M2.GND@14, M2.GND@15, M2.GND@16, M2.GND@17, M2.GND@2, M2.GND@3, M2.GND@4, M2.GND@5, M2.GND@7, M2.GND@8, R15.1, R2.1, S1.5, U12.GND, U13.GND, U2.AGND, U2.PGND, U5.GND
- net P4_RX: now also C5.2, R1.1, R3.1; no longer C31.2, R42.1, R43.1
- net P4_RX_N: now also J8.P6, M1.P4_RX-, R1.2; no longer J3.8, J6.3, R43.2
- net P4_RX_P: now also J8.P3, M1.P4_RX+, R3.2; no longer J3.7, J6.2, R42.2
- net P4_TX: now also C2.2, R2.1, R8.1; no longer C32.2, R44.1, R45.1
- net P4_TX_N: now also J8.P2, M1.P4_TX-, R8.2; no longer J3.2, J6.5, R45.2
- net P4_TX_P: now also J8.P1, M1.P4_TX+, R2.2; no longer J3.1, J6.4, R44.2
- net SHIELD: now also C13.2, C3.2, J8.P8, J8.SHIELD@1, J8.SHIELD@2; no longer C34.2, J3.6, J3.SHIELD@1, J3.SHIELD@2
- net USB_N: now also M1.USB_N; no longer M2.USB-
- net USB_P: now also M1.USB_P; no longer M2.USB+
Other:
- note removed: "/"
- note removed: "Antenna"
- note removed: "Core"
- note removed: "JUMPSTART SWITCH"
- note removed: "Jumpstart"
- note removed: "LEDS"
- note removed: "POWER"
- note removed: "PoE"
- note removed: "PolyFuse"
- note removed: "Power Supply"
- note removed: "WIRELESS"
- moved on the sheet: BOARD1, C1, C10, C11, C12, C13, C14, C18, C2, C22, C23, C24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
