File: Domino Qi Mini/Domino Qi Mini No Teardrop.sch (EAGLE design)
At the start: 90 parts, among them J1 MH22-1, J2 MH22-1, M1 DOMINO, Q1 AP2302GN, Q2 2SC4081, SW1 IT-1210, SW2 IT-1210, SW3 IT-1210, U1 MP65151DJ, U2 ATMEGA32U4-AU/MU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

Commit message: Domino Qi Mini Rev. C: changed NTB0102GU to NTB0102GF
Parts:
- U5: value NTB0102GU -> NTB0102GF; device Domino:NTB0102GU -> Domino:NTB0102GF; PARTNO NTB0102GU -> NTB0102GF
Changed lines of the file:
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@@
 <attribute name="DATABASE" value="./../Common/BOM/Domino_DB.txt"/>
 <attribute name="DRAWN" value="M.STEMPIN"/>
-<attribute name="REV" value="B"/>
+<attribute name="REV" value="C"/>
 </attributes>
 <variantdefs>
@@
 <attribute name="PARTNO" value="NTB0104GU12"/>
 </part>
-<part name="U5" library="Domino" deviceset="NTB0102" device="GU">
-<attribute name="PARTNO" value="NTB0102GU"/>
+<part name="U5" library="Domino" deviceset="NTB0102" device="GF" value="NTB0102GF">
+<attribute name="PARTNO" value="NTB0102GF"/>
 </part>
 <part name="U6" library="Domino" deviceset="MAX3375E" device="EKA+T">

Commit message: Domino Qi Mini Rev. D: corrected bridge pinout
Connections:
- net MISO: now also U4.B3; no longer U4.B4
- net MOSI: now also U4.B2; no longer U4.B3
- net SCK: now also U4.B4; no longer U4.B2
Changed lines of the file:
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@@
 <attribute name="DATABASE" value="./../Common/BOM/Domino_DB.txt"/>
 <attribute name="DRAWN" value="M.STEMPIN"/>
-<attribute name="REV" value="C"/>
+<attribute name="REV" value="D"/>
 </attributes>
 <variantdefs>
@@
 <net name="SS" class="0">
 <segment>
-<pinref part="U2" gate="G$1" pin="(SS/PCINT0)PB0"/>
-<wire x1="121.92" y1="154.94" x2="149.86" y2="154.94" width="0.1524" layer="91"/>
-<label x="144.78" y="154.94" size="1.778" layer="95"/>
+<wire x1="142.24" y1="154.94" x2="149.86" y2="154.94" width="0.1524" layer="91"/>
+<label x="142.24" y="154.94" size="1.778" layer="95"/>
 <pinref part="U4" gate="G$1" pin="B1"/>
 </segment>
@@
 <pinref part="J2" gate="G$1" pin="16"/>
 </segment>
+<segment>
+<pinref part="U2" gate="G$1" pin="(SS/PCINT0)PB0"/>
+<wire x1="121.92" y1="154.94" x2="134.62" y2="154.94" width="0.1524" layer="91"/>
+<label x="134.62" y="154.94" size="1.778" layer="95" rot="MR0"/>
+</segment>
 </net>
 <net name="SCK" class="0">
 <segment>
-<pinref part="U2" gate="G$1" pin="(SCLK/PCINT1)PB1"/>
-<wire x1="149.86" y1="152.4" x2="121.92" y2="152.4" width="0.1524" layer="91"/>
-<label x="144.78" y="152.4" size="1.778" layer="95"/>
-<pinref part="U4" gate="G$1" pin="B2"/>
+<wire x1="149.86" y1="147.32" x2="142.24" y2="147.32" width="0.1524" layer="91"/>
+<label x="142.24" y="147.32" size="1.778" layer="95"/>
+<pinref part="U4" gate="G$1" pin="B4"/>
 </segment>
 <segment>
@@
 <pinref part="J2" gate="G$1" pin="14"/>
 </segment>
+<segment>
+<pinref part="U2" gate="G$1" pin="(SCLK/PCINT1)PB1"/>
+<wire x1="134.62" y1="152.4" x2="121.92" y2="152.4" width="0.1524" layer="91"/>
+<label x="134.62" y="152.4" size="1.778" layer="95" rot="MR0"/>
+</segment>
 </net>
 <net name="MOSI" class="0">
 <segment>
-<pinref part="U2" gate="G$1" pin="(PDI/MOSI/PCINT2)PB2"/>
-<wire x1="121.92" y1="149.86" x2="149.86" y2="149.86" width="0.1524" layer="91"/>
-<label x="144.78" y="149.86" size="1.778" layer="95"/>
-<pinref part="U4" gate="G$1" pin="B3"/>
+<wire x1="142.24" y1="152.4" x2="149.86" y2="152.4" width="0.1524" layer="91"/>
+<label x="142.24" y="152.4" size="1.778" layer="95"/>
+<pinref part="U4" gate="G$1" pin="B2"/>
 </segment>
 <segment>
@@
 <pinref part="J2" gate="G$1" pin="15"/>
 </segment>
-</net>
-<net name="MISO" class="0">
-<segment>
-<pinref part="U2" gate="G$1" pin="(PD0/MISO/PCINT3)PB3"/>
-<wire x1="149.86" y1="147.32" x2="121.92" y2="147.32" width="0.1524" layer="91"/>
-<label x="144.78" y="147.32" size="1.778" layer="95"/>
-<pinref part="U4" gate="G$1" pin="B4"/>
-</segment>
 <segment>
-<wire x1="297.18" y1="45.72" x2="297.18" y2="55.88" width="0.1524" layer="91"/>
-<label x="297.18" y="45.72" size="1.778" layer="95" rot="R90"/>
-<pinref part="J2" gate="G$1" pin="17"/>
+<pinref part="U2" gate="G$1" pin="(PDI/MOSI/PCINT2)PB2"/>
+<wire x1="121.92" y1="149.86" x2="134.62" y2="149.86" width="0.1524" layer="91"/>
+<label x="134.62" y="149.86" size="1.778" layer="95" rot="MR0"/>
 </segment>
 </net>
@@
 </segment>
 </net>
+<net name="MISO" class="0">
+<segment>
+<wire x1="149.86" y1="149.86" x2="142.24" y2="149.86" width="0.1524" layer="91"/>
+<label x="142.24" y="149.86" size="1.778" layer="95"/>
+<pinref part="U4" gate="G$1" pin="B3"/>
+</segment>
+<segment>
+<pinref part="U2" gate="G$1" pin="(PD0/MISO/PCINT3)PB3"/>
+<wire x1="134.62" y1="147.32" x2="121.92" y2="147.32" width="0.1524" layer="91"/>
+<label x="134.62" y="147.32" size="1.778" layer="95" rot="MR0"/>
+</segment>
+<segment>
+<wire x1="297.18" y1="45.72" x2="297.18" y2="55.88" width="0.1524" layer="91"/>
+<label x="297.18" y="45.72" size="1.778" layer="95" rot="R90"/>
+<pinref part="J2" gate="G$1" pin="17"/>
+</segment>
+</net>
